File: indikator.kicad_sch (KiCad schematic)
At the start: 101 parts, among them Q1 AO3400A, Q10 AO3400A, Q11 AO3400A, Q12 AO3400A, Q13 AO3400A, Q14 AO3400A, Q15 AO3400A, Q16 AO3400A, Q17 AO3400A, Q18 AO3400A, Q19 AO3400A, Q2 AO3400A, Q20 AO3400A, Q21 AO3400A, Q22 AO3400A, Q23 AO3400A, Q24 AO3400A, Q3 AO3400A, Q4 AO3400A, Q5 AO3400A, Q6 AO3400A, Q7 AO3400A, Q8 AO3400A, Q9 AO3400A, U1 XIAO-ESP32-C3-SMD, U2 74HC595, U3 74HC595, U4 74HC595

Commit message: add capacitors for the 74hc595s
Parts:
- added C1, C2, C3: C, Package_SO:SOIC-8_3.9x4.9mm_P1.27mm, symbol Device:C
Connections:
- net ESP3V3: now also U3.10 (~{SRCLR}), U3.16 (VCC), U4.10 (~{SRCLR}), U4.16 (VCC), C1.1, C2.1, C3.1
- net GND: now also C1.2, C2.2, C3.2
- net SRCLK: now reaches U3.11 (SRCLK)
- net SRCLK: now also U1.6 (D5), U2.11 (SRCLK), U4.11 (SRCLK)
- net RCLK: now reaches U3.12 (RCLK)
- net RCLK: now also U1.5 (D4), U2.12 (RCLK), U4.12 (RCLK)
- net QH'1: now reaches U3.14 (SER)
- net QH'1: now also U2.9 (QH')
- net QH'2: now reaches U3.9 (QH')
- net QH'2: now also U4.14 (SER)
- net SER: now reaches U1.7 (D6)
- net SER: now also U2.14 (SER)
Other:
- moved on the sheet: BT1, U1

Commit message: finish schematics
Parts:
- removed BT1: Battery, symbol Device:Battery
- added J1: Conn_01x02, Package_SO:SOIC-8_3.9x4.9mm_P1.27mm, symbol Connector_Generic:Conn_01x02
Connections:
- net GND: now also U1.22 (GND), J1.2 (Pin_2)
- net VBAT+: now also U1.21 (VBAT), J1.1 (Pin_1)
Other:
- moved on the sheet: C1, C2, C3, D1, D10, D11, D12, D13, D14, D15, D16, D17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

Commit message: fix all the erc warnings
Connections:
- no-connect marks 0 -> 17
Other:
- moved on the sheet: C1, C2, C3, D1, D10, D11, D12, D13, D14, D15, D16, D17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

Commit message: connect footprints
Parts:
- C1, C2, C3: footprint Package_SO:SOIC-8_3.9x4.9mm_P1.27mm -> Capacitor_SMD:C_0805_2012Metric
- D1, D10, D11, D12, D13, D14, D15, D16, D17, D18, D19, D2, D20, D21, D22, D23, D24, D3, D4, D5, D6, D7, D8, D9: footprint (none) -> LED_SMD:LED_0805_2012Metric
- J1: footprint Package_SO:SOIC-8_3.9x4.9mm_P1.27mm -> Connector_JST:JST_XH_B2B-XH-AM_1x02_P2.50mm_Vertical
- R1, R10, R11, R12, R13, R14, R15, R16, R17, R18, R19, R2, R20, R21, R22, R23, R24, R25, R26, R27, R28, R29, R3, R30, R31, R32, R33, R34, R35, R36, R37, R38, R39, R4, R40, R41, R42, R43, R44, R45, R46, R47, R48, R5, R6, R7, R8, R9: footprint Package_SO:SOJ-36_10.16x23.495mm_P1.27mm -> Resistor_SMD:R_0805_2012Metric
- U1: footprint Seeed_Studio_XIAO_Series:XIAO-ESP32-C3-SMD -> RF_Module:MCU_Seeed_ESP32C3
- U2, U3, U4: footprint Package_CSP:Xilinx_CSG48_7.0x7.0mm_Layout7x7_P0.8mm -> Package_DIP:DIP-16_W7.62mm
