File: _restore_backup_2026-09-28T05-52-07-289/indikator.kicad_pcb (KiCad board)
At the start: 2 copper layers, 125 x 52.5 mm, 104 parts, among them J1 Conn_01x02, Q1 AO3400A, Q10 AO3400A, Q11 AO3400A, Q12 AO3400A, Q13 AO3400A, Q14 AO3400A, Q15 AO3400A, Q16 AO3400A, Q17 AO3400A, Q18 AO3400A, Q19 AO3400A, Q2 AO3400A, Q20 AO3400A, Q21 AO3400A, Q22 AO3400A, Q23 AO3400A, Q24 AO3400A, Q3 AO3400A, Q4 AO3400A, Q5 AO3400A, Q6 AO3400A, Q7 AO3400A, Q8 AO3400A, Q9 AO3400A, U1 XIAO-ESP32-C3-SMD, U2 74HC595, U3 74HC595, U4 74HC595

Commit message: ROUTING IS FRICKIN IMPOSSIBLE BRUH
Parts:
- moved U4 238.6 mm to (50.5, 22.5), turned to 0 degrees
- moved C3 209.8 mm to (35.0, 111.0)
- moved C2 194.1 mm to (36.5, 103.5)
- moved U1 143.3 mm to (117.5, 87.6)
- moved Q21 141.6 mm to (276.4, 29.4), turned to 0 degrees
- moved R41 140.1 mm to (275.9, 19.5)
- moved C1 139.1 mm to (42.0, 109.0)
- moved R42 135.8 mm to (275.9, 22.4)
- moved R39 128.0 mm to (266.9, 19.5)
- moved R37 127.1 mm to (258.0, 19.6)
- moved U3 124.9 mm to (37.0, 22.5)
- moved R40 123.3 mm to (266.9, 22.4)
- moved R38 122.4 mm to (258.0, 22.5)
- moved Q20 118.4 mm to (267.4, 28.9), turned to 0 degrees
- moved Q19 113.0 mm to (258.1, 30.0), turned to 0 degrees
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Connections:
- R2 pad 1: Net-(Q1-D) -> Net-(D1-K)
- R2 pad 2: Net-(D1-K) -> Net-(Q1-D)
- R25 pad 1: Net-(Q9-D) -> Net-(D9-K)
- R25 pad 2: Net-(D9-K) -> Net-(Q9-D)
- R41 pad 1: Net-(Q17-D) -> Net-(D17-K)
- R41 pad 2: Net-(D17-K) -> Net-(Q17-D)
Routing:
- net Net-(Q13-G): track 81.2 -> 0.00 mm
- net Net-(Q4-G): track 48.2 -> 0.00 mm
- net Net-(Q10-G): track 41.6 -> 0.00 mm
- net Net-(Q3-G): track 40.2 -> 0.00 mm
- net Net-(Q8-G): track 35.4 -> 0.00 mm
- net Net-(Q11-G): track 35.3 -> 0.00 mm
- net Net-(Q7-G): track 32.1 -> 0.00 mm
- net Net-(Q2-G): track 30.2 -> 0.00 mm
- net Net-(Q6-G): track 29.8 -> 0.00 mm
- net Net-(Q12-G): track 29.0 -> 0.00 mm
- net Net-(Q5-G): track 26.4 -> 0.00 mm
- net GND: track 24.6 -> 0.00 mm
- net Net-(Q1-G): track 21.2 -> 0.00 mm
- net Net-(D9-K): track 4.77 -> 0.00 mm
- net Net-(D8-K): track 4.77 -> 0.00 mm
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Other:
- board outline removed
