File: _restore_backup_2026-09-28T08-22-44-731/indikator.kicad_pcb (KiCad board)
At the start: 2 copper layers, 125 x 52.5 mm, 104 parts, among them J1 Conn_01x02, Q1 AO3400A, Q10 AO3400A, Q11 AO3400A, Q12 AO3400A, Q13 AO3400A, Q14 AO3400A, Q15 AO3400A, Q16 AO3400A, Q17 AO3400A, Q18 AO3400A, Q19 AO3400A, Q2 AO3400A, Q20 AO3400A, Q21 AO3400A, Q22 AO3400A, Q23 AO3400A, Q24 AO3400A, Q3 AO3400A, Q4 AO3400A, Q5 AO3400A, Q6 AO3400A, Q7 AO3400A, Q8 AO3400A, Q9 AO3400A, U1 XIAO-ESP32-C3-SMD, U2 74HC595, U3 74HC595, U4 74HC595

Commit message: ROUTING IS FRICKIN IMPOSSIBLE BRUH
Parts:
- moved U3 132.0 mm to (200.4, 157.6), turned to 90 degrees
- moved Q12 70.5 mm to (185.7, 82.0), turned to 0 degrees
- moved Q11 67.5 mm to (177.6, 82.0), turned to 0 degrees
- moved Q10 64.7 mm to (169.6, 82.0), turned to 0 degrees
- moved Q9 61.7 mm to (161.1, 82.0), turned to 0 degrees
- moved R17 60.1 mm to (159.1, 77.6), turned to 0 degrees
- moved R18 60.1 mm to (163.1, 77.6), turned to 0 degrees
- moved R19 60.1 mm to (167.1, 77.6), turned to 0 degrees
- moved R20 60.1 mm to (171.1, 77.6), turned to 0 degrees
- moved Q17 59.0 mm to (129.7, 93.5), turned to 0 degrees
- moved R33 58.9 mm to (127.7, 89.1), turned to 0 degrees
- moved R34 58.9 mm to (131.7, 89.1), turned to 0 degrees
- moved R35 58.9 mm to (135.7, 89.1), turned to 0 degrees
- moved R36 58.9 mm to (139.7, 89.1), turned to 0 degrees
- moved Q20 58.7 mm to (153.7, 93.5), turned to 0 degrees
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Connections:
- R2 pad 1: Net-(Q1-D) -> Net-(D1-K)
- R2 pad 2: Net-(D1-K) -> Net-(Q1-D)
- R25 pad 1: Net-(Q9-D) -> Net-(D9-K)
- R25 pad 2: Net-(D9-K) -> Net-(Q9-D)
- R41 pad 1: Net-(Q17-D) -> Net-(D17-K)
- R41 pad 2: Net-(D17-K) -> Net-(Q17-D)
Routing:
- net Net-(Q13-G): track 81.2 -> 0.00 mm
- net Net-(Q4-G): track 48.2 -> 0.00 mm
- net Net-(Q10-G): track 41.6 -> 0.00 mm
- net Net-(Q3-G): track 40.2 -> 0.00 mm
- net Net-(Q8-G): track 35.4 -> 0.00 mm
- net Net-(Q11-G): track 35.3 -> 0.00 mm
- net Net-(Q7-G): track 32.1 -> 0.00 mm
- net Net-(Q2-G): track 30.2 -> 0.00 mm
- net Net-(Q6-G): track 29.8 -> 0.00 mm
- net Net-(Q12-G): track 29.0 -> 0.00 mm
- net Net-(Q5-G): track 26.4 -> 0.00 mm
- net GND: track 24.6 -> 0.00 mm
- net Net-(Q1-G): track 21.2 -> 0.00 mm
- net Net-(D9-K): track 4.77 -> 0.00 mm
- net Net-(D8-K): track 4.77 -> 0.00 mm
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